Commit message: pushing whatever changes there are to the old SVD repo on my laptop at the moment

File: src/realsense-ros/realsense2_description/tests/dual_d435.xacro (robot description, xacro)
@@ -3,9 +3,9 @@
   <xacro:include filename="../urdf/_d435.urdf.xacro" />
   <xacro:arg name="use_nominal_extrinsics" default="True" />
-  <link name="realsense_frame" />
-  <xacro:sensor_d435 parent="realsense_frame" name="camera_bottom">
+  <link name="base_link" />
+  <xacro:sensor_d435 parent="base_link" name="camera_bottom">
     <origin xyz="0 0 0" rpy="0 0 0"/>
   </xacro:sensor_d435>
-  <xacro:sensor_d435 parent="realsense_frame" name="camera_top">
+  <xacro:sensor_d435 parent="base_link" name="camera_top">
     <origin xyz="0 0 0.2" rpy="0 0 0"/>
   </xacro:sensor_d435>

File: src/realsense-ros/realsense2_description/tests/one_of_each.xacro (robot description, xacro)
@@ -10,5 +10,5 @@
     <origin xyz="0 0 0" rpy="0 0 0"/>
   </xacro:sensor_d415>
-  <xacro:sensor_d435 parent="realsense_frame" name="d435">
+  <xacro:sensor_d435 parent="base_link" name="d435">
     <origin xyz="0 0 0.1" rpy="0 0 0"/>
   </xacro:sensor_d435>

File: src/realsense-ros/realsense2_description/urdf/test_d435_camera.urdf.xacro (robot description, xacro)
@@ -5,6 +5,6 @@
   <xacro:arg name="use_mesh" default="true" />
   <xacro:include filename="$(find realsense2_description)/urdf/_d435.urdf.xacro" />
-  <link name="realsense_frame" />
-  <xacro:sensor_d435 parent="realsense_frame" use_nominal_extrinsics="$(arg use_nominal_extrinsics)" add_plug="$(arg add_plug)" use_mesh="$(arg use_mesh)">
+  <link name="base_link" />
+  <xacro:sensor_d435 parent="base_link" use_nominal_extrinsics="$(arg use_nominal_extrinsics)" add_plug="$(arg add_plug)" use_mesh="$(arg use_mesh)">
     <origin xyz="0 0 0" rpy="0 0 0"/>
   </xacro:sensor_d435>

File: src/realsense-ros/realsense2_description/urdf/test_d435i_camera.urdf.xacro (robot description, xacro)
@@ -3,6 +3,6 @@
   <xacro:arg name="use_nominal_extrinsics" default="false" />
   <xacro:include filename="$(find realsense2_description)/urdf/_d435i.urdf.xacro"/>
-  <link name="realsense_frame" />
-  <xacro:sensor_d435i parent="realsense_frame" use_nominal_extrinsics="$(arg use_nominal_extrinsics)">
+  <link name="base_link" />
+  <xacro:sensor_d435i parent="base_link" use_nominal_extrinsics="$(arg use_nominal_extrinsics)">
     <origin xyz="0 0 0" rpy="0 0 0"/>
   </xacro:sensor_d435i>
